File: MysensorsDimmer.brd (EAGLE design)
At the start: 64.7 x 64.7 mm, 56 parts, among them IC1 7805DT, IC2 AT25DF512C-SSHN-B, IC3 ATSHA204A, IC4 DS1820, J1 22-27-2021-02, J2 22-27-2021-02, J3 22-27-2021-02, J4 22-27-2021-02, J5 22-27-2021-02, Q1 IRF530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

Commit message: modifications after v1.0 version (see changelog.txt)
Parts:
- C2: device SparkFun-Passives:0603-CAP -> SparkFun-Passives:1206
- moved C2 4.34 mm to (15.7, 53.5)
- moved X1 0.50 mm to (60.3, 29.6)
- moved X2 0.50 mm to (4.60, 31.6)
- moved X3 0.50 mm to (34.3, 4.70)
Connections:
- new net D8: ARDUINO1.8, IC2.1, R2.1
- net A5: no longer IC2.1, R2.1
- net VCC: now also ISP.2
Routing:
- net D8: track 0.00 -> 37.4 mm, vias 0 -> 3
- net VCC: track 52.3 -> 73.6 mm, vias 1 -> 3
- net A5: track 8.30 -> 0.00 mm
- net GND: track 285.6 -> 291.2 mm
- net N$2: track 0.00 -> 3.06 mm
- net D5: track 6.82 -> 8.57 mm
- net RST: track 39.1 -> 40.5 mm
- net 12V: track 51.8 -> 53.1 mm
- net 5V: track 183.7 -> 184.9 mm
- net N$22: track 13.3 -> 13.9 mm
- net A3: track 22.5 -> 23.0 mm
- net N$10: track 13.3 -> 13.8 mm
- net A2: track 24.3 -> 24.8 mm
- net N$26: track 7.20 -> 7.71 mm
- net N$27: track 7.18 -> 7.68 mm
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Other:
- board text added: "MySensors Dimmer v1.1"
- board text removed: "MySensors Dimmer v1.0"
